Commit message: Dexhand improvements and correction for mid and pinky fingers, improved README, position controlled for testing.

File: config/dexhand.ros2_control.xacro (robot description, xacro)
@@ -10,145 +10,148 @@
             <joint name="wrist_pitch_lower">
                 <command_interface name="position"/>
-                <command_interface name="velocity"/>
-                <command_interface name="effort"/>
                 <state_interface name="position">
                   <param name="initial_value">${initial_positions['wrist_pitch_lower']}</param>
                 </state_interface>
+                <state_interface name="velocity"/>
             </joint>
             <joint name="wrist_yaw">
                 <command_interface name="position"/>
-                <command_interface name="velocity"/>
-                <command_interface name="effort"/>
                 <state_interface name="position">
                   <param name="initial_value">${initial_positions['wrist_yaw']}</param>
                 </state_interface>
+                <state_interface name="velocity"/>
             </joint>
             <joint name="index_yaw">
                 <command_interface name="position"/>
-                <command_interface name="velocity"/>
-                <command_interface name="effort"/>
                 <state_interface name="position">
                   <param name="initial_value">${initial_positions['index_yaw']}</param>
                 </state_interface>
+                <state_interface name="velocity"/>
             </joint>
             <joint name="index_pitch">
                 <command_interface name="position"/>
-                <command_interface name="velocity"/>
-                <command_interface name="effort"/>
                 <state_interface name="position">
                   <param name="initial_value">${initial_positions['index_pitch']}</param>
                 </state_interface>
+                <state_interface name="velocity"/>
             </joint>
             <joint name="index_knuckle">
                 <command_interface name="position"/>
-                <command_interface name="velocity"/>
-                <command_interface name="effort"/>
                 <state_interface name="position">
                   <param name="initial_value">${initial_positions['index_knuckle']}</param>
                 </state_interface>
+                <state_interface name="velocity"/>
             </joint>
             <joint name="index_tip">
                 <command_interface name="position"/>
-                <command_interface name="velocity"/>
-                <command_interface name="effort"/>
                 <state_interface name="position">
                   <param name="initial_value">${initial_positions['index_tip']}</param>
                 </state_interface>
+                <state_interface name="velocity"/>
             </joint>
             <joint name="middle_yaw">
                 <command_interface name="position"/>
-                <command_interface name="velocity"/>
-                <command_interface name="effort"/>
                 <state_interface name="position">
                   <param name="initial_value">${initial_positions['middle_yaw']}</param>
                 </state_interface>
+                <state_interface name="velocity"/>
             </joint>
             <joint name="middle_pitch">
                 <command_interface name="position"/>
-                <command_interface name="velocity"/>
-                <command_interface name="effort"/>
                 <state_interface name="position">
                   <param name="initial_value">${initial_positions['middle_pitch']}</param>
                 </state_interface>
+                <state_interface name="velocity"/>
             </joint>
             <joint name="middle_knuckle">
                 <command_interface name="position"/>
-                <command_interface name="velocity"/>
-                <command_interface name="effort"/>
                 <state_interface name="position">
                   <param name="initial_value">${initial_positions['middle_knuckle']}</param>
                 </state_interface>
+                <state_interface name="velocity"/>
             </joint>
             <joint name="middle_tip">
                 <command_interface name="position"/>
-                <command_interface name="velocity"/>
-                <command_interface name="effort"/>
                 <state_interface name="position">
                   <param name="initial_value">${initial_positions['middle_tip']}</param>
                 </state_interface>
+                <state_interface name="velocity"/>
+            </joint>
+            <joint name="ring_pitch">
+                <command_interface name="position"/>
+                <state_interface name="position">
+                  <param name="initial_value">${initial_positions['ring_pitch']}</param>
+                </state_interface>
+                <state_interface name="velocity"/>
+            </joint>
+            <joint name="ring_knuckle">
+                <command_interface name="position"/>
+                <state_interface name="position">
+                  <param name="initial_value">${initial_positions['ring_knuckle']}</param>
+                </state_interface>
+                <state_interface name="velocity"/>
+            </joint>
+            <joint name="ring_tip">
+                <command_interface name="position"/>
+                <state_interface name="position">
+                  <param name="initial_value">${initial_positions['ring_tip']}</param>
+                </state_interface>
+                <state_interface name="velocity"/>
             </joint>
             <joint name="pinky_yaw">
                 <command_interface name="position"/>
-                <command_interface name="velocity"/>
-                <command_interface name="effort"/>
                 <state_interface name="position">
                   <param name="initial_value">${initial_positions['pinky_yaw']}</param>
                 </state_interface>
+                <state_interface name="velocity"/>
             </joint>
             <joint name="pinky_pitch">
                 <command_interface name="position"/>
-                <command_interface name="velocity"/>
-                <command_interface name="effort"/>
                 <state_interface name="position">
                   <param name="initial_value">${initial_positions['pinky_pitch']}</param>
                 </state_interface>
+                <state_interface name="velocity"/>
             </joint>
             <joint name="pinky_knuckle">
                 <command_interface name="position"/>
-                <command_interface name="velocity"/>
-                <command_interface name="effort"/>
                 <state_interface name="position">
                   <param name="initial_value">${initial_positions['pinky_knuckle']}</param>
                 </state_interface>
+                <state_interface name="velocity"/>
             </joint>
             <joint name="pinky_tip">
                 <command_interface name="position"/>
-                <command_interface name="velocity"/>
-                <command_interface name="effort"/>
                 <state_interface name="position">
                   <param name="initial_value">${initial_positions['pinky_tip']}</param>
                 </state_interface>
+                <state_interface name="velocity"/>
             </joint>
             <joint name="thumb_roll">
                 <command_interface name="position"/>
-                <command_interface name="velocity"/>
-                <command_interface name="effort"/>
                 <state_interface name="position">
                   <param name="initial_value">${initial_positions['thumb_roll']}</param>
                 </state_interface>
+                <state_interface name="velocity"/>
             </joint>
             <joint name="thumb_pitch">
                 <command_interface name="position"/>
-                <command_interface name="velocity"/>
-                <command_interface name="effort"/>
                 <state_interface name="position">
                   <param name="initial_value">${initial_positions['thumb_pitch']}</param>
                 </state_interface>
+                <state_interface name="velocity"/>
             </joint>
             <joint name="thumb_knuckle">
                 <command_interface name="position"/>
-                <command_interface name="velocity"/>
-                <command_interface name="effort"/>
                 <state_interface name="position">
                   <param name="initial_value">${initial_positions['thumb_knuckle']}</param>
                 </state_interface>
+                <state_interface name="velocity"/>
             </joint>
             <joint name="thumb_tip">
                 <command_interface name="position"/>
-                <command_interface name="velocity"/>
-                <command_interface name="effort"/>
                 <state_interface name="position">
                   <param name="initial_value">${initial_positions['thumb_tip']}</param>
                 </state_interface>
+                <state_interface name="velocity"/>
             </joint>
         </ros2_control>
